File: hardware/hardware.sch (KiCad schematic (older format))
At the start: 23 parts, among them J1 DIN-5_180degree, U1 Teensy3.2, U2 TeensyAudioShield3.2, U3 6N138

Commit message: Use correct schematic diagram for RGB led
Parts:
- D2: symbol Device:LED_RGBC -> Device:LED_RCGB
Other:
- moved on the sheet: R4, R5
Changed lines of the file:
@@
 	9255 4695 9255 4545
 $Comp
-L Device:LED_RGBC D2
+L Device:LED_RCGB D2
 U 1 1 5FCC987F
 P 4800 5550
@@
 NoConn ~ 2300 1625
 Wire Wire Line
-	5000 5750 5100 5750
+	5000 5550 5100 5550
 Wire Wire Line
-	5600 5750 5400 5750
-Text Label 5600 5750 0    50   ~ 0
+	5600 5550 5400 5550
+Text Label 5600 5550 0    50   ~ 0
 RGB_G
 $Comp
 L Device:R R4
 U 1 1 5FCD0BCE
+P 5250 5550
+F 0 "R4" V 5043 5550 50  0000 C CNN
+F 1 "220" V 5134 5550 50  0000 C CNN
+F 2 "Resistor_THT:R_Axial_DIN0207_L6.3mm_D2.5mm_P10.16mm_Horizontal" V 5180 5550 50  0001 C CNN
+F 3 "~" H 5250 5550 50  0001 C CNN
+	1    5250 5550
+	0    1    1    0
+$EndComp
+$Comp
+L power:GND #PWR0131
+U 1 1 5FCDFF2C
+P 4500 5550
+F 0 "#PWR0131" H 4500 5300 50  0001 C CNN
+F 1 "GND" V 4505 5422 50  0000 R CNN
+F 2 "" H 4500 5550 50  0001 C CNN
+F 3 "" H 4500 5550 50  0001 C CNN
+	1    4500 5550
+	0    1    1    0
+$EndComp
+Wire Wire Line
+	5400 5750 5600 5750
+Text Label 5600 5750 0    50   ~ 0
+RGB_B
+$Comp
+L Device:R R5
+U 1 1 5FCD61B6
 P 5250 5750
-F 0 "R4" V 5043 5750 50  0000 C CNN
+F 0 "R5" V 5043 5750 50  0000 C CNN
 F 1 "220" V 5134 5750 50  0000 C CNN
 F 2 "Resistor_THT:R_Axial_DIN0207_L6.3mm_D2.5mm_P10.16mm_Horizontal" V 5180 5750 50  0001 C CNN
@@
 $EndComp
 Wire Wire Line
-	5200 5550 5000 5550
-$Comp
-L power:GND #PWR0131
-U 1 1 5FCDFF2C
-P 5200 5550
-F 0 "#PWR0131" H 5200 5300 50  0001 C CNN
-F 1 "GND" V 5205 5422 50  0000 R CNN
-F 2 "" H 5200 5550 50  0001 C CNN
-F 3 "" H 5200 5550 50  0001 C CNN
-	1    5200 5550
-	0    -1   -1   0
-$EndComp
-Wire Wire Line
-	4200 5550 4000 5550
-Text Label 4000 5550 2    50   ~ 0
-RGB_B
-$Comp
-L Device:R R5
-U 1 1 5FCD61B6
-P 4350 5550
-F 0 "R5" V 4143 5550 50  0000 C CNN
-F 1 "220" V 4234 5550 50  0000 C CNN
-F 2 "Resistor_THT:R_Axial_DIN0207_L6.3mm_D2.5mm_P10.16mm_Horizontal" V 4280 5550 50  0001 C CNN
-F 3 "~" H 4350 5550 50  0001 C CNN
-	1    4350 5550
-	0    -1   -1   0
-$EndComp
+	5000 5750 5100 5750
 $EndSCHEMATC
